File: MDBT.sch (KiCad schematic (older format))
At the start: 6 parts, among them P2 CONN_01X03, U3 MDBT40

Commit message: 2017年10月29日
Parts:
- P2: footprint connectors:Socket_Strip_Straight_1x03_Pitch2.54mm -> connectors:Socket_Strip_Straight_1x04_Pitch2.54mm; symbol CONN_01X03 -> CONN_01X04
Connections:
- new net GPIO5: P2.4 (P4)
Changed lines of the file:
@@
 	6750 2650 7600 2650
 $Comp
-L CONN_01X03 P2
+L CONN_01X04 P2
 U 1 1 59966FFB
 P 7800 4100
 F 0 "P2" H 7800 4300 50  0000 C CNN
 F 1 "CONN_01X03" V 7900 4100 50  0000 C CNN
-F 2 "connectors:Socket_Strip_Straight_1x03_Pitch2.54mm" H 7800 4100 50  0001 C CNN
+F 2 "connectors:Socket_Strip_Straight_1x04_Pitch2.54mm" H 7800 4100 50  0001 C CNN
 F 3 "" H 7800 4100 50  0001 C CNN
 	1    7800 4100
@@
 	6750 2850 7300 2850
 Wire Wire Line
-	7300 2850 7300 4000
-Wire Wire Line
-	7300 4000 7600 4000
-Wire Wire Line
 	6750 2950 7200 2950
 Wire Wire Line
-	7200 2950 7200 4100
+	7300 2850 7300 3950
 Wire Wire Line
-	7200 4100 7600 4100
+	7300 3950 7600 3950
 Wire Wire Line
-	7450 4650 7450 4200
+	7600 4050 7200 4050
 Wire Wire Line
-	7450 4200 7600 4200
+	7200 4050 7200 2950
+Wire Wire Line
+	7600 4150 7450 4150
+Wire Wire Line
+	7450 4150 7450 4650
+Wire Wire Line
+	7600 4250 7550 4250
+Wire Wire Line
+	7550 4250 7550 4400
+Text HLabel 7550 4400 3    60   BiDi ~ 0
+GPIO5
 $EndSCHEMATC
