File: led.sch (KiCad schematic (older format))
At the start: 122 parts, among them Q1 MOS_P

Commit message: Chicory init commit from Daisy
Parts:
- LED1, LED10, LED11, LED12, LED13, LED14, LED15, LED16, LED17, LED18, LED19, LED2, LED20, LED21, LED22, LED23, LED24, LED25, LED26, LED27, LED28, LED29, LED3, LED30, LED31, LED32, LED33, LED34, LED35, LED36, LED37, LED38, LED38_625, LED39, LED4, LED40, LED41, LED42, LED5, LED6, LED7, LED8, LED9: symbol LED -> LED-RESCUE-keyboard
- R4: footprint resistors:R_0805 -> resistors:R_0805_V1
